File: instrumental_integrator/instrumental_integrator.kicad_sch (KiCad schematic)
At the start: 61 parts, among them CN2 282841-2, CN3 282841-2, J10 Conn_01x01_Socket, J12 Conn_01x01_Socket, J13 Conn_01x01_Socket, J14 Conn_01x01_Socket, J15 Conn_01x01_Socket, J16 Conn_01x01_Socket, J4 Conn_01x01_Socket, J5 Conn_01x01_Socket, J6 Conn_01x01_Socket, J7 Conn_01x01_Socket, J8 Conn_01x01_Socket, J9 Conn_01x01_Socket, Q1 2N7002, SW2 TS1603-TZ38HBM, U1 INA828IDR, U10 ADS8681RUM, U11 SS12D10G5, U12 SS12D10G5, U2 C3D22UF500V82CB0300, U3 C3D22UF500V82CB0300, U4 BAT54_C2926171, U5 BAT54_C2926171, U6 BAT54_C2926171, U7 BAT54_C2926171, U9 TLV2387DR

Commit message: finished pcb design V1
Parts:
- C9: footprint Capacitor_SMD:C_0805_2012Metric -> Capacitor_SMD:C_0603_1608Metric
Changed lines of the file:
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@@
 			)
 		)
-		(property "Footprint" "Capacitor_SMD:C_0805_2012Metric"
+		(property "Footprint" "Capacitor_SMD:C_0603_1608Metric"
 			(at 251.1552 96.52 0)
 			(hide yes)
